Commit message: [feat] Changed from position controllers to velocity controllers in simulation

File: crane_plus_simulation/urdf/simulated_crane_plus.urdf.xacro (robot description, xacro)
@@ -8,6 +8,12 @@
   <!-- Include the Crane+ generator macro -->
   <xacro:include filename="$(find crane_plus_description)/urdf/crane_plus.xacro"/>
+    <!-- Used for fixing robot to Gazebo 'base_link' -->
+  <link name="world"/>
   <!-- Link to provide the location reference for the arm -->
-  <link name="base_link"/>
+   <link name="base_link"/>
+  <joint name="fixed" type="fixed">
+    <parent link="world"/>
+    <child link="base_link"/>
+  </joint>
   <!-- Use the crane_plus macro to configure a Crane+ arm with desired joint
        velocities limit and lower/upper limits for the first joint. This
@@ -26,8 +32,8 @@
     <type>transmission_interface/SimpleTransmission</type>
     <joint name="crane_plus_shoulder_revolute_joint">
-      <hardwareInterface>hardware_interface/PositionJointInterface</hardwareInterface>
+      <hardwareInterface>hardware_interface/VelocityJointInterface</hardwareInterface>
     </joint>
     <actuator name="shoulder_revolute_servo">
-      <hardwareInterface>PositionJointInterface</hardwareInterface>
+      <hardwareInterface>VelocityJointInterface</hardwareInterface>
       <mechanicalReduction>1</mechanicalReduction>
     </actuator>
@@ -37,8 +43,8 @@
     <type>transmission_interface/SimpleTransmission</type>
     <joint name="crane_plus_shoulder_flex_joint">
-      <hardwareInterface>hardware_interface/PositionJointInterface</hardwareInterface>
+      <hardwareInterface>hardware_interface/VelocityJointInterface</hardwareInterface>
     </joint>
     <actuator name="shoulder_flex_servo">
-      <hardwareInterface>PositionJointInterface</hardwareInterface>
+      <hardwareInterface>VelocityJointInterface</hardwareInterface>
       <mechanicalReduction>1</mechanicalReduction>
     </actuator>
@@ -48,8 +54,8 @@
     <type>transmission_interface/SimpleTransmission</type>
     <joint name="crane_plus_elbow_joint">
-      <hardwareInterface>hardware_interface/PositionJointInterface</hardwareInterface>
+      <hardwareInterface>hardware_interface/VelocityJointInterface</hardwareInterface>
     </joint>
     <actuator name="elbow_servo">
-      <hardwareInterface>PositionJointInterface</hardwareInterface>
+      <hardwareInterface>VelocityJointInterface</hardwareInterface>
       <mechanicalReduction>1</mechanicalReduction>
     </actuator>
@@ -59,8 +65,8 @@
     <type>transmission_interface/SimpleTransmission</type>
     <joint name="crane_plus_wrist_joint">
-      <hardwareInterface>hardware_interface/PositionJointInterface</hardwareInterface>
+      <hardwareInterface>hardware_interface/VelocityJointInterface</hardwareInterface>
     </joint>
     <actuator name="wrist_servo">
-      <hardwareInterface>PositionJointInterface</hardwareInterface>
+      <hardwareInterface>VelocityJointInterface</hardwareInterface>
       <mechanicalReduction>1</mechanicalReduction>
     </actuator>
@@ -78,6 +84,9 @@
   </transmission>
   <gazebo>
-    <plugin name="control" filename="libgazebo_ros_control.so"/>
+    <plugin name="control" filename="libgazebo_ros_control.so">
+		<robotSimType>gazebo_ros_control/DefaultRobotHWSim</robotSimType>
+	</plugin>
     <plugin name="joint_state_publisher" filename="libgazebo_ros_joint_state_publisher.so">
+    <updateRate>100.0</updateRate>
       <jointName>
         crane_plus_shoulder_revolute_joint,

Commit message: [feat] Added control.launch with updated gazebo settings

File: crane_plus_simulation/urdf/simulated_crane_plus.urdf.xacro (robot description, xacro)
@@ -1,15 +1,14 @@
 <?xml version="1.0"?>
-<robot
-    name="crane_plus"
-    xmlns:xacro="http://ros.org/wiki/xacro"
-    xmlns:sensor="http://playerstage.sourceforge.net/gazebo/xmlschema/#sensor"
-    xmlns:controller="http://playerstage.sourceforge.net/gazebo/xmlschema/#controller"
-    xmlns:interface="http://playerstage.sourceforge.net/gazebo/xmlschema/#interface">
+<robot name="crane_plus"
+  xmlns:xacro="http://ros.org/wiki/xacro"
+  xmlns:sensor="http://playerstage.sourceforge.net/gazebo/xmlschema/#sensor"
+  xmlns:controller="http://playerstage.sourceforge.net/gazebo/xmlschema/#controller"
+  xmlns:interface="http://playerstage.sourceforge.net/gazebo/xmlschema/#interface">
   <!-- Include the Crane+ generator macro -->
   <xacro:include filename="$(find crane_plus_description)/urdf/crane_plus.xacro"/>
-    <!-- Used for fixing robot to Gazebo 'base_link' -->
+  <!-- Used for fixing robot to Gazebo 'base_link' -->
   <link name="world"/>
   <!-- Link to provide the location reference for the arm -->
-   <link name="base_link"/>
+  <link name="base_link"/>
   <joint name="fixed" type="fixed">
     <parent link="world"/>
@@ -20,8 +19,5 @@
        allows accessing different operational areas, e.g. left-handed vs.
        right-handed robots. -->
-  <crane_plus parent="base_link"
-              servo_color="black" bracket_color="grey" gripper_color="black"
-              joints_vlimit="1.571"
-              pan_llimit="-2.617" pan_ulimit="2.617">
+  <crane_plus parent="base_link" servo_color="black" bracket_color="grey" gripper_color="black" joints_vlimit="1.571" pan_llimit="-2.617" pan_ulimit="2.617">
     <!-- Place the "floating" arm at the origin of the base_link. -->
     <origin xyz="0 0 0"/>
@@ -85,8 +81,8 @@
   <gazebo>
     <plugin name="control" filename="libgazebo_ros_control.so">
-		<robotSimType>gazebo_ros_control/DefaultRobotHWSim</robotSimType>
-	</plugin>
+      <robotSimType>gazebo_ros_control/DefaultRobotHWSim</robotSimType>
+    </plugin>
     <plugin name="joint_state_publisher" filename="libgazebo_ros_joint_state_publisher.so">
-    <updateRate>100.0</updateRate>
+      <updateRate>100.0</updateRate>
       <jointName>
         crane_plus_shoulder_revolute_joint,
